File: KiCad/mb486sr.kicad_pcb (KiCad board)
At the start: 2 copper layers, 170.2 x 243.8 mm, 45 parts, among them J301 Conn_SIMM72, J302 Conn_SIMM72, P1 POWER_SW, P2 RESET, P3 POWER, P4 SERIAL, P5 SERIAL, P6 RESET, P7 POWER_LED, SW1 POWER, SW2 RESET, U1 Intel_P24T

Commit message: Version 0.3: Update DRAM schematic, pull-ups/pull-downs, CPU configuration jumpers
Signed-off-by: Sergey Kiselev <skiselev@gmail.com>
Connections:
- net /~PS_ON renamed /~{PS_ON}
Routing:
- net /~{0WS}: track 0.00 -> 75.3 mm
- net /~0WS: track 75.3 -> 0.00 mm
Other:
- net class Default removed
- net class Power removed
- board text added: "Motherboard 486 Sandy River - Version 1.0 Copyright (C) 2022 Sergey Kiselev"
- board text removed: "Motherboard 486 White River - Version 1.0 Copyright (C) 2022 Sergey Kiselev"
